File: Schematics_and_Layouts/Zuendbox_v3/Zuendbox_v3.kicad_pcb (KiCad board)
At the start: 2 copper layers, 160 x 100 mm, 141 parts, among them J1 USB_B, J2 AVR-ISP-10, Q1 IRF3708, Q10 IRF3708, Q11 IRF3708, Q12 IRF3708, Q13 IRF3708, Q14 IRF3708, Q15 IRF3708, Q16 IRF3708, Q17 BC327, Q18 BC337, Q19 IRF4905, Q2 IRF3708, Q20 BC327, Q21 BC337, Q3 IRF3708, Q4 IRF3708, Q5 IRF3708, Q6 IRF3708, Q7 IRF3708, Q8 IRF3708, Q9 IRF3708, U1 DM13A, U10 DS18B20, U2 MCP6002-xP, U3 RFM69CW-RF_Module, U4 ATmega328P-PU, U5 74HC595, U6 XL6009_Module, U7 LM1084-3.3, U8 74HC595, U9 MCP2221_IP, Y1 Crystal

Commit message: Manual update
Parts:
- R1: value 33k -> 47k
Changed lines of the file:
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@@
-(kicad_pcb (version 20171130) (host pcbnew "(6.0.0-rc1-dev-402-g020d837de)")
+(kicad_pcb (version 20171130) (host pcbnew "(6.0.0-rc1-dev-508-gaf2dcd61b)")
   (general
     (thickness 1.6)
@@
     (pad_drill 1.2)
     (pad_to_mask_clearance 0.2)
+    (solder_mask_min_width 0.25)
     (aux_axis_origin 65.135 44.635)
     (grid_origin 65.135 144.635)
@@
       (effects (font (size 0.8 0.8) (thickness 0.16)))
     )
-    (fp_text value 33k (at 5.08 2.37 270) (layer F.Fab)
+    (fp_text value 47k (at 5.08 2.37 270) (layer F.Fab)
       (effects (font (size 0.8 0.8) (thickness 0.16)))
     )
